Commit message: Added updated tests.

File: examples/ugv.urdf (robot description, URDF)
Before this commit: robot UGV, 5 links, 4 joints
Links:
- removed link chassis
- removed link front_left_wheel_body
- removed link front_right_wheel_body
- removed link rear_left_wheel_body
- removed link rear_right_wheel_body
- added link UGV_chassis; visual box size=0.1 0.16 0.04
- added link UGV_front_left_wheel_0_extensioni_body; visual box size=0.008333333333333333 0.01 0.01
- added link UGV_front_left_wheel_1_extensioni_body; visual box size=0.008333333333333333 0.01 0.01
- added link UGV_front_left_wheel_2_extensioni_body; visual box size=0.008333333333333333 0.01 0.01
- added link UGV_front_left_wheel_body; visual cylinder length=0.01 radius=0.025
- added link UGV_front_right_wheel_0_extensioni_body; visual box size=0.008333333333333333 0.01 0.01
- added link UGV_front_right_wheel_1_extensioni_body; visual box size=0.008333333333333333 0.01 0.01
- added link UGV_front_right_wheel_2_extensioni_body; visual box size=0.008333333333333333 0.01 0.01
- added link UGV_front_right_wheel_body; visual cylinder length=0.01 radius=0.025
- added link UGV_rear_left_wheel_0_extensioni_body; visual box size=0.008333333333333333 0.01 0.01
- added link UGV_rear_left_wheel_1_extensioni_body; visual box size=0.008333333333333333 0.01 0.01
- added link UGV_rear_left_wheel_2_extensioni_body; visual box size=0.008333333333333333 0.01 0.01
- added link UGV_rear_left_wheel_body; visual cylinder length=0.01 radius=0.025
- added link UGV_rear_right_wheel_0_extensioni_body; visual box size=0.008333333333333333 0.01 0.01
- added link UGV_rear_right_wheel_1_extensioni_body; visual box size=0.008333333333333333 0.01 0.01
- added link UGV_rear_right_wheel_2_extensioni_body; visual box size=0.008333333333333333 0.01 0.01
- added link UGV_rear_right_wheel_body; visual cylinder length=0.01 radius=0.025
Joints:
- removed joint front_left_wheel_joint
- removed joint front_right_wheel_joint
- removed joint rear_left_wheel_joint
- removed joint rear_right_wheel_joint
- added joint UGV_front_left_wheel_0_extensioni_joint: type revolute, parent UGV_front_left_wheel_body, child UGV_front_left_wheel_0_extensioni_body, limit effort=0 velocity=0
- added joint UGV_front_left_wheel_1_extensioni_joint: type revolute, parent UGV_front_left_wheel_body, child UGV_front_left_wheel_1_extensioni_body, limit effort=0 velocity=0
- added joint UGV_front_left_wheel_2_extensioni_joint: type revolute, parent UGV_front_left_wheel_body, child UGV_front_left_wheel_2_extensioni_body, limit effort=0 velocity=0
- added joint UGV_front_left_wheel_joint: type revolute, parent UGV_chassis, child UGV_front_left_wheel_body, origin xyz=0.05 -0.085 0 rpy=0 0 0, axis 0 1 0, limit effort=0 velocity=0
- added joint UGV_front_right_wheel_0_extensioni_joint: type revolute, parent UGV_front_right_wheel_body, child UGV_front_right_wheel_0_extensioni_body, limit effort=0 velocity=0
- added joint UGV_front_right_wheel_1_extensioni_joint: type revolute, parent UGV_front_right_wheel_body, child UGV_front_right_wheel_1_extensioni_body, limit effort=0 velocity=0
- added joint UGV_front_right_wheel_2_extensioni_joint: type revolute, parent UGV_front_right_wheel_body, child UGV_front_right_wheel_2_extensioni_body, limit effort=0 velocity=0
- added joint UGV_front_right_wheel_joint: type revolute, parent UGV_chassis, child UGV_front_right_wheel_body, origin xyz=0.05 0.085 0 rpy=0 0 0, axis 0 1 0, limit effort=0 velocity=0
- added joint UGV_rear_left_wheel_0_extensioni_joint: type revolute, parent UGV_rear_left_wheel_body, child UGV_rear_left_wheel_0_extensioni_body, limit effort=0 velocity=0
- added joint UGV_rear_left_wheel_1_extensioni_joint: type revolute, parent UGV_rear_left_wheel_body, child UGV_rear_left_wheel_1_extensioni_body, limit effort=0 velocity=0
- added joint UGV_rear_left_wheel_2_extensioni_joint: type revolute, parent UGV_rear_left_wheel_body, child UGV_rear_left_wheel_2_extensioni_body, limit effort=0 velocity=0
- added joint UGV_rear_left_wheel_joint: type revolute, parent UGV_chassis, child UGV_rear_left_wheel_body, origin xyz=-0.05 -0.085 0 rpy=0 0 0, axis 0 1 0, limit effort=0 velocity=0
- added joint UGV_rear_right_wheel_0_extensioni_joint: type revolute, parent UGV_rear_right_wheel_body, child UGV_rear_right_wheel_0_extensioni_body, limit effort=0 velocity=0
- added joint UGV_rear_right_wheel_1_extensioni_joint: type revolute, parent UGV_rear_right_wheel_body, child UGV_rear_right_wheel_1_extensioni_body, limit effort=0 velocity=0
- added joint UGV_rear_right_wheel_2_extensioni_joint: type revolute, parent UGV_rear_right_wheel_body, child UGV_rear_right_wheel_2_extensioni_body, limit effort=0 velocity=0
- added joint UGV_rear_right_wheel_joint: type revolute, parent UGV_chassis, child UGV_rear_right_wheel_body, origin xyz=-0.05 0.085 0 rpy=0 0 0, axis 0 1 0, limit effort=0 velocity=0

Commit message: Added collision and inertial blocks.

File: examples/ugv.urdf (robot description, URDF)
Before this commit: robot UGV, 17 links, 16 joints
Links:
- removed link UGV_front_left_wheel_0_extensioni_body
- removed link UGV_front_left_wheel_1_extensioni_body
- removed link UGV_front_left_wheel_2_extensioni_body
- removed link UGV_front_right_wheel_0_extensioni_body
- removed link UGV_front_right_wheel_1_extensioni_body
- removed link UGV_front_right_wheel_2_extensioni_body
- removed link UGV_rear_left_wheel_0_extensioni_body
- removed link UGV_rear_left_wheel_1_extensioni_body
- removed link UGV_rear_left_wheel_2_extensioni_body
- removed link UGV_rear_right_wheel_0_extensioni_body
- removed link UGV_rear_right_wheel_1_extensioni_body
- removed link UGV_rear_right_wheel_2_extensioni_body
- added link UGV_front_left_wheel_0_extension_body, mass 0.0008333333333333333; collision box size=0.008333333333333333 0.01 0.01; visual box size=0.008333333333333333 0.01 0.01
- added link UGV_front_left_wheel_1_extension_body, mass 0.0008333333333333333; collision box size=0.008333333333333333 0.01 0.01; visual box size=0.008333333333333333 0.01 0.01
- added link UGV_front_left_wheel_2_extension_body, mass 0.0008333333333333333; collision box size=0.008333333333333333 0.01 0.01; visual box size=0.008333333333333333 0.01 0.01
- added link UGV_front_right_wheel_0_extension_body, mass 0.0008333333333333333; collision box size=0.008333333333333333 0.01 0.01; visual box size=0.008333333333333333 0.01 0.01
- added link UGV_front_right_wheel_1_extension_body, mass 0.0008333333333333333; collision box size=0.008333333333333333 0.01 0.01; visual box size=0.008333333333333333 0.01 0.01
- added link UGV_front_right_wheel_2_extension_body, mass 0.0008333333333333333; collision box size=0.008333333333333333 0.01 0.01; visual box size=0.008333333333333333 0.01 0.01
- added link UGV_rear_left_wheel_0_extension_body, mass 0.0008333333333333333; collision box size=0.008333333333333333 0.01 0.01; visual box size=0.008333333333333333 0.01 0.01
- added link UGV_rear_left_wheel_1_extension_body, mass 0.0008333333333333333; collision box size=0.008333333333333333 0.01 0.01; visual box size=0.008333333333333333 0.01 0.01
- added link UGV_rear_left_wheel_2_extension_body, mass 0.0008333333333333333; collision box size=0.008333333333333333 0.01 0.01; visual box size=0.008333333333333333 0.01 0.01
- added link UGV_rear_right_wheel_0_extension_body, mass 0.0008333333333333333; collision box size=0.008333333333333333 0.01 0.01; visual box size=0.008333333333333333 0.01 0.01
- added link UGV_rear_right_wheel_1_extension_body, mass 0.0008333333333333333; collision box size=0.008333333333333333 0.01 0.01; visual box size=0.008333333333333333 0.01 0.01
- added link UGV_rear_right_wheel_2_extension_body, mass 0.0008333333333333333; collision box size=0.008333333333333333 0.01 0.01; visual box size=0.008333333333333333 0.01 0.01
- link UGV_chassis: mass None -> 0.64; geometry collision box size=0.1 0.16 0.04; visual box size=0.1 0.16 0.04
- link UGV_front_left_wheel_body: mass None -> 0.01963495408493621; geometry collision cylinder length=0.01 radius=0.025; visual cylinder length=0.01 radius=0.025
- link UGV_front_right_wheel_body: mass None -> 0.01963495408493621; geometry collision cylinder length=0.01 radius=0.025; visual cylinder length=0.01 radius=0.025
- link UGV_rear_left_wheel_body: mass None -> 0.01963495408493621; geometry collision cylinder length=0.01 radius=0.025; visual cylinder length=0.01 radius=0.025
- link UGV_rear_right_wheel_body: mass None -> 0.01963495408493621; geometry collision cylinder length=0.01 radius=0.025; visual cylinder length=0.01 radius=0.025
Joints:
- removed joint UGV_front_left_wheel_0_extensioni_joint
- removed joint UGV_front_left_wheel_1_extensioni_joint
- removed joint UGV_front_left_wheel_2_extensioni_joint
- removed joint UGV_front_right_wheel_0_extensioni_joint
- removed joint UGV_front_right_wheel_1_extensioni_joint
- removed joint UGV_front_right_wheel_2_extensioni_joint
- removed joint UGV_rear_left_wheel_0_extensioni_joint
- removed joint UGV_rear_left_wheel_1_extensioni_joint
- removed joint UGV_rear_left_wheel_2_extensioni_joint
- removed joint UGV_rear_right_wheel_0_extensioni_joint
- removed joint UGV_rear_right_wheel_1_extensioni_joint
- removed joint UGV_rear_right_wheel_2_extensioni_joint
- added joint UGV_front_left_wheel_0_extension_joint: type revolute, parent UGV_front_left_wheel_body, child UGV_front_left_wheel_0_extension_body, limit effort=0 velocity=0
- added joint UGV_front_left_wheel_1_extension_joint: type revolute, parent UGV_front_left_wheel_body, child UGV_front_left_wheel_1_extension_body, limit effort=0 velocity=0
- added joint UGV_front_left_wheel_2_extension_joint: type revolute, parent UGV_front_left_wheel_body, child UGV_front_left_wheel_2_extension_body, limit effort=0 velocity=0
- added joint UGV_front_right_wheel_0_extension_joint: type revolute, parent UGV_front_right_wheel_body, child UGV_front_right_wheel_0_extension_body, limit effort=0 velocity=0
- added joint UGV_front_right_wheel_1_extension_joint: type revolute, parent UGV_front_right_wheel_body, child UGV_front_right_wheel_1_extension_body, limit effort=0 velocity=0
- added joint UGV_front_right_wheel_2_extension_joint: type revolute, parent UGV_front_right_wheel_body, child UGV_front_right_wheel_2_extension_body, limit effort=0 velocity=0
- added joint UGV_rear_left_wheel_0_extension_joint: type revolute, parent UGV_rear_left_wheel_body, child UGV_rear_left_wheel_0_extension_body, limit effort=0 velocity=0
- added joint UGV_rear_left_wheel_1_extension_joint: type revolute, parent UGV_rear_left_wheel_body, child UGV_rear_left_wheel_1_extension_body, limit effort=0 velocity=0
- added joint UGV_rear_left_wheel_2_extension_joint: type revolute, parent UGV_rear_left_wheel_body, child UGV_rear_left_wheel_2_extension_body, limit effort=0 velocity=0
- added joint UGV_rear_right_wheel_0_extension_joint: type revolute, parent UGV_rear_right_wheel_body, child UGV_rear_right_wheel_0_extension_body, limit effort=0 velocity=0
- added joint UGV_rear_right_wheel_1_extension_joint: type revolute, parent UGV_rear_right_wheel_body, child UGV_rear_right_wheel_1_extension_body, limit effort=0 velocity=0
- added joint UGV_rear_right_wheel_2_extension_joint: type revolute, parent UGV_rear_right_wheel_body, child UGV_rear_right_wheel_2_extension_body, limit effort=0 velocity=0
- joint UGV_front_left_wheel_joint: origin xyz=0.05 -0.085 0 rpy=0 0 0 -> xyz=0.05 -0.085 0
- joint UGV_front_right_wheel_joint: origin xyz=0.05 0.085 0 rpy=0 0 0 -> xyz=0.05 0.085 0
- joint UGV_rear_left_wheel_joint: origin xyz=-0.05 -0.085 0 rpy=0 0 0 -> xyz=-0.05 -0.085 0
- joint UGV_rear_right_wheel_joint: origin xyz=-0.05 0.085 0 rpy=0 0 0 -> xyz=-0.05 0.085 0
